File: PCB_Files/card_dealer_pcb/card_dealer_pcb.kicad_sch (KiCad schematic)
At the start: 0 parts

Commit message: Added PCB schematics
Parts:
- added C1: 2,2uf, Package_TO_SOT_SMD:SOT-23-6, symbol Device:C
- added D1, D2, D3: D, Diode_THT:D_5W_P10.16mm_Horizontal, symbol Device:D
- added J1, J2: Conn_01x20_Pin, Connector_PinHeader_2.54mm:PinHeader_1x20_P2.54mm_Vertical, symbol Connector:Conn_01x20_Pin
- added J10: IR_Sensor_8, Connector_PinHeader_2.54mm:PinHeader_1x03_P2.54mm_Vertical, symbol Connector:Conn_01x03_Pin
- added J11: IR_Sensor_7, Connector_PinHeader_2.54mm:PinHeader_1x03_P2.54mm_Vertical, symbol Connector:Conn_01x03_Pin
- added J12: L298N, Package_TO_SOT_THT:TO-220-15_P2.54x5.08mm_StaggerOdd_Lead4.58mm_Vertical, symbol Connector:Conn_01x04_Pin
- added J3: Barrel_Jack, Connector:Tag-Connect_TC2030-IDC-FP_2x03_P1.27mm_Vertical, symbol Connector:Barrel_Jack
- added J4: IR_Sensor_1, Connector_PinHeader_2.54mm:PinHeader_1x03_P2.54mm_Vertical, symbol Connector:Conn_01x03_Pin
- added J5: IR_Sensor_2, Connector_PinHeader_2.54mm:PinHeader_1x03_P2.54mm_Vertical, symbol Connector:Conn_01x03_Pin
- added J6: IR_Sensor_4, Connector_PinHeader_2.54mm:PinHeader_1x03_P2.54mm_Vertical, symbol Connector:Conn_01x03_Pin
- added J7: IR_Sensor_5, Connector_PinHeader_2.54mm:PinHeader_1x03_P2.54mm_Vertical, symbol Connector:Conn_01x03_Pin
- added J8: IR_Sensor_3, Connector_PinHeader_2.54mm:PinHeader_1x03_P2.54mm_Vertical, symbol Connector:Conn_01x03_Pin
- added J9: IR_Sensor_6, Connector_PinHeader_2.54mm:PinHeader_1x03_P2.54mm_Vertical, symbol Connector:Conn_01x03_Pin
- added M1, M2, M3: Motor_DC, Connector_PinHeader_1.00mm:PinHeader_1x02_P1.00mm_Vertical, symbol Motor:Motor_DC
- added Q1, Q2, Q3: IRLZ44N, Package_TO_SOT_THT:TO-220-3_Vertical, symbol Transistor_FET:IRLZ44N
- added R1, R4, R6: 10K, Resistor_THT:R_Axial_DIN0411_L9.9mm_D3.6mm_P12.70mm_Horizontal, symbol Device:R
- added R2, R3, R5: 100, Resistor_THT:R_Axial_DIN0411_L9.9mm_D3.6mm_P12.70mm_Horizontal, symbol Device:R
Connections:
- new net: D1.2 (A), M1.2 (-), Q1.2 (D)
- new net: D3.2 (A), M3.2 (-), Q3.2 (D)
- new net: D2.2 (A), M2.2 (-), Q2.2 (D)
- new net 3V3: J1.1 (Pin_1), J2.3 (Pin_3)
- new net 5V: C1.1, D1.1 (K), D2.1 (K), D3.1 (K), J1.3 (Pin_3), J10.3 (Pin_3), J11.3 (Pin_3), J2.1 (Pin_1), J3.1, J4.3 (Pin_3), J5.3 (Pin_3), J6.3 (Pin_3), J7.3 (Pin_3), J8.3 (Pin_3), J9.3 (Pin_3), M1.1 (+), M2.1 (+), M3.1 (+), Q1.1 (G), Q2.1 (G), Q3.1 (G), R1.1, R2.2, R3.2, R4.1, R5.2, R6.1
- new net GNDREF: C1.2, J1.2 (Pin_2), J10.2 (Pin_2), J11.2 (Pin_2), J2.2 (Pin_2), J3.2, J4.2 (Pin_2), J5.2 (Pin_2), J6.2 (Pin_2), J7.2 (Pin_2), J8.2 (Pin_2), J9.2 (Pin_2), Q1.3 (S), Q2.3 (S), Q3.3 (S), R1.2, R4.2, R6.2
- new net PA0: J2.15 (Pin_15), R2.1
- new net PA1: J2.14 (Pin_14), R3.1
- new net PA10: J1.14 (Pin_14)
- new net PA11: J1.13 (Pin_13)
- new net PA12: J1.12 (Pin_12)
- new net PA15: J1.11 (Pin_11)
- new net PA2: J2.13 (Pin_13), R5.1
- new net PA3: J12.EN1 (Pin_1), J2.12 (Pin_12)
- new net PA4: J12.EN2 (Pin_2), J2.11 (Pin_11)
- new net PA5: J12.EN3 (Pin_3), J2.10 (Pin_10)
- new net PA6: J12.EN4 (Pin_4), J2.9 (Pin_9)
- new net PA7: J2.8 (Pin_8)
- new net PA8: J1.16 (Pin_16)
- new net PA9: J1.15 (Pin_15)
- new net PB0: J2.7 (Pin_7)
- new net PB1: J2.6 (Pin_6)
- new net PB10: J10.1 (Pin_1), J2.4 (Pin_4)
- new net PB12: J1.20 (Pin_20)
- new net PB13: J1.19 (Pin_19)
- new net PB14: J1.18 (Pin_18)
- new net PB15: J1.17 (Pin_17)
- new net PB2: J2.5 (Pin_5)
- new net PB3: J1.10 (Pin_10), J4.1 (Pin_1)
- new net PB4: J1.9 (Pin_9), J5.1 (Pin_1)
- new net PB5: J1.8 (Pin_8), J8.1 (Pin_1)
- new net PB6: J1.7 (Pin_7), J6.1 (Pin_1)
- new net PB7: J1.6 (Pin_6), J7.1 (Pin_1)
- new net PB8: J1.5 (Pin_5), J9.1 (Pin_1)
- new net PB9: J1.4 (Pin_4), J11.1 (Pin_1)
- new net PC13: J2.19 (Pin_19)
- new net PC14: J2.18 (Pin_18)
- new net PC15: J2.17 (Pin_17)
- new net R: J2.16 (Pin_16)
- new net VBAT: J2.20 (Pin_20)
Other:
- note added: "DC Motors"
- note added: "IR Sensors"
- note added: "L298N"
- note added: "Power In"
- note added: "STM32 Blackpill"
- company: (none) -> Emin Akman
- title: (none) -> Main PCB

Commit message: Changed the pcb schematics
Parts:
- added C2, C3, C4: 470uF, symbol Device:C
- added C5, C6: 10uf, Package_TO_SOT_SMD:SOT-23-6, symbol Device:C
- C1: value 2,2uf -> 2200uf
Connections:
- net 5V: now also C2.2, C3.2, C4.2, C5.1, C6.1
- net GNDREF renamed GND
- net GND: now also C2.1, C3.1, C4.1, C5.2, C6.2
