File: PCB_Files/card_dealer_remote/card_dealer_remote.kicad_sch (KiCad schematic)
At the start: 9 parts, among them SW1 SW_Push, U1 TLC555xD

Commit message: Changed the pcb schematics
Parts:
- added Q1: 2N2219, Package_TO_SOT_THT:TO-39-3, symbol Transistor_BJT:2N2219
- added R4: 33, Package_DIP:DIP-8_W7.62mm, symbol Device:R
- R3: value 100 -> 1K
Connections:
- net GNDREF: now also Q1.1 (E); no longer D1.2 (A)
- net at D1.1 (K): now also Q1.3 (C); no longer R3.2
- net at R1.1, SW1.1, U1.4 (~{RST})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: now also R4.1
- new net: D1.2 (A), R4.2
- new net: Q1.2 (B), R3.2
Other:
- moved on the sheet: D1

Commit message: made cad files for remote
Parts:
- C1, C2: footprint Package_SO:SOIC-8_3.9x4.9mm_P1.27mm -> Capacitor_THT:CP_Radial_D5.0mm_P2.00mm
- R1, R2: footprint Package_DIP:DIP-8_W7.62mm -> Resistor_THT:R_Axial_DIN0207_L6.3mm_D2.5mm_P7.62mm_Horizontal
- R3: value 1K -> 4.7K; footprint Package_DIP:DIP-8_W7.62mm -> Resistor_THT:R_Axial_DIN0207_L6.3mm_D2.5mm_P7.62mm_Horizontal
- R4: value 33 -> 100; footprint Package_DIP:DIP-8_W7.62mm -> Resistor_THT:R_Axial_DIN0207_L6.3mm_D2.5mm_P7.62mm_Horizontal
- U1: footprint Package_SO:SOIC-8_3.9x4.9mm_P1.27mm -> Package_DIP:DIP-8_W7.62mm
Changed lines of the file:
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@@
 			)
 		)
-		(property "Value" "1K"
+		(property "Value" "4.7K"
 			(at 90.932 70.104 90)
 			(show_name no)
@@
 			)
 		)
-		(property "Footprint" "Package_DIP:DIP-8_W7.62mm"
+		(property "Footprint" "Resistor_THT:R_Axial_DIN0207_L6.3mm_D2.5mm_P7.62mm_Horizontal"
 			(at 92.71 67.818 90)
 			(hide yes)
@@
 			)
 		)
-		(property "Footprint" "Package_DIP:DIP-8_W7.62mm"
+		(property "Footprint" "Resistor_THT:R_Axial_DIN0207_L6.3mm_D2.5mm_P7.62mm_Horizontal"
 			(at 56.642 52.07 90)
 			(hide yes)
@@
 			)
 		)
-		(property "Footprint" "Package_SO:SOIC-8_3.9x4.9mm_P1.27mm"
+		(property "Footprint" "Package_DIP:DIP-8_W7.62mm"
 			(at 73.66 90.17 0)
 			(hide yes)
@@
 			)
 		)
-		(property "Value" "33"
+		(property "Value" "100"
 			(at 89.662 48.514 90)
 			(show_name no)
@@
 			)
 		)
-		(property "Footprint" "Package_DIP:DIP-8_W7.62mm"
+		(property "Footprint" "Resistor_THT:R_Axial_DIN0207_L6.3mm_D2.5mm_P7.62mm_Horizontal"
 			(at 91.44 46.228 90)
 			(hide yes)
@@
 			)
 		)
-		(property "Footprint" "Package_SO:SOIC-8_3.9x4.9mm_P1.27mm"
+		(property "Footprint" "Capacitor_THT:CP_Radial_D5.0mm_P2.00mm"
 			(at 88.5952 78.74 0)
 			(hide yes)
@@
 			)
 		)
-		(property "Footprint" "Package_SO:SOIC-8_3.9x4.9mm_P1.27mm"
+		(property "Footprint" "Capacitor_THT:CP_Radial_D5.0mm_P2.00mm"
 			(at 54.3052 81.28 0)
 			(hide yes)
@@
 			)
 		)
-		(property "Footprint" "Package_DIP:DIP-8_W7.62mm"
+		(property "Footprint" "Resistor_THT:R_Axial_DIN0207_L6.3mm_D2.5mm_P7.62mm_Horizontal"
 			(at 51.562 67.31 90)
 			(hide yes)
